File: PaneledKit/PaneledKit.kicad_pcb (KiCad board)
At the start: 2 copper layers, 62.2 x 94.4 mm, 202 parts, among them IC1 MCF8316A1VRGFR, IC1 VNH7100BASTR, IC2 TJA1050T_CM, IC3 LSM6DS3TR-C, IC4 TMC2209-LA, J1 SM04B-SRSS-TB, J10 Conn_01x02_Pin, J11 Conn_01x06_Pin, J12 Conn_01x02_Pin, J13 Conn_01x02_Pin, J14 Conn_01x02_Pin, J15 Conn_01x02_Pin, J2 SM04B-SRSS-TB, J3 Conn_01x03_Pin, J3 TS02-66-60-BK-160-LCR-D, J3 XT30PB, J4 TS02-66-60-BK-160-LCR-D, J4 XT30PB, J5 SM04B-SRSS-TB, J6 SM04B-SRSS-TB, J7 TS02-66-60-BK-160-LCR-D, J7 XT30PB, J8 Conn_01x03_Pin, J9 TS02-66-60-BK-160-LCR-D, Q1 BSS138, Q2 BSS138, SW1 DSHP04TJGER, U1 MOUDLE-SEEEDUINO-XIAO-ESP32C3, U2 DM-OLED096-636

Commit message: DaisyBoardOut
Parts:
- added C16: 100nF 50V, Capacitor_SMD:C_0402_1005Metric, F.Cu at (101.6, 40.4)
- added C17: 1uF 50V, Capacitor_SMD:C_0402_1005Metric, F.Cu at (107.2, 40.4)
- added C18: 1uF 50V, Capacitor_SMD:C_0402_1005Metric, F.Cu at (103.6, 40.4)
- added C19: 100nF 50V, Capacitor_SMD:C_0402_1005Metric, F.Cu at (109.2, 40.4)
- added C20: 100nF 50V, Capacitor_SMD:C_0402_1005Metric, F.Cu at (107.8, 52.7)
- added C21: 1uF 50V, Capacitor_SMD:C_0402_1005Metric, F.Cu at (107.8, 50.8)
- added C22: 100nF 50V, Capacitor_SMD:C_0402_1005Metric, F.Cu at (108.2, 56.9)
- added C23: 30pF, Capacitor_SMD:C_0402_1005Metric, F.Cu at (98.8, 55.9)
- added C24: 30pF, Capacitor_SMD:C_0402_1005Metric, F.Cu at (99.6, 60.8)
- added C25: 1uF 50V, Capacitor_SMD:C_0402_1005Metric, F.Cu at (120.1, 56.7)
- added C26: 100nF 50V, Capacitor_SMD:C_0402_1005Metric, F.Cu at (120.1, 54.7)
- added C32: 100nF 50V, Capacitor_SMD:C_0402_1005Metric, F.Cu at (110.2, 67.1)
- added C33: 100nF 50V, Capacitor_SMD:C_0402_1005Metric, F.Cu at (118.0, 67.4)
- added D3: KT-0603R, LED_SMD:LED_0603_1608Metric, F.Cu at (94.2, 33.3)
- added D5: SS34, Diode_SMD:D_SOD-123, F.Cu at (97.0, 42.2)
- added DR1: COS4427SR, Package_SO:SOP-8_3.76x4.96mm_P1.27mm, F.Cu at (103.4, 51.3)
- added DR2: COS4427SR, Package_SO:SOP-8_3.76x4.96mm_P1.27mm, F.Cu at (107.4, 44.7)
- added DR3: COS4427SR, Package_SO:SOP-8_3.76x4.96mm_P1.27mm, F.Cu at (101.9, 44.7)
- added DR4: COS4427SR, Package_SO:SOP-8_3.76x4.96mm_P1.27mm, F.Cu at (115.8, 55.6)
- added IC5: TJA1050T_CM, SamacSys_Parts:SOIC127P600X175-8N, F.Cu at (103.5, 56.9)
- added IC8: LSM6DS3TR-C, SamacSys_Parts:LSM6DS3USTR, F.Cu at (114.4, 68.1)
- added J15: SM04B-SRSS-TB, Connector_JST:JST_SH_SM04B-SRSS-TB_1x04-1MP_P1.00mm_Horizontal, F.Cu at (95.8, 51.9)
- added J17: SM04B-SRSS-TB, Connector_JST:JST_SH_SM04B-SRSS-TB_1x04-1MP_P1.00mm_Horizontal, F.Cu at (95.8, 60.1)
- added J18: Conn_01x04_Pin, TerminalBlock:TerminalBlock_Xinya_XY308-2.54-4P_1x04_P2.54mm_Horizontal, F.Cu at (119.6, 43.2)
- added J19: Conn_01x03_Pin, Connector_PinHeader_2.54mm:PinHeader_1x03_P2.54mm_Vertical, F.Cu at (121.4, 59.5)
- added J36: SM04B-SRSS-TB, Connector_JST:JST_SH_SM04B-SRSS-TB_1x04-1MP_P1.00mm_Horizontal, F.Cu at (96.7, 68.1)
- added J37: SM04B-SRSS-TB, Connector_JST:JST_SH_SM04B-SRSS-TB_1x04-1MP_P1.00mm_Horizontal, F.Cu at (105.1, 68.1)
- added J7: XT30PB, JST_Sorted:XT30PB, F.Cu at (107.7, 36.2)
- added J8: XT30PB, Library:Xt30 Horizontal, F.Cu at (102.3, 36.3)
- added J9: Conn_01x04_Pin, TerminalBlock:TerminalBlock_Xinya_XY308-2.54-4P_1x04_P2.54mm_Horizontal, F.Cu at (119.6, 28.5)
- added JP12: SolderJumper_2_Open, Jumper:SolderJumper-2_P1.3mm_Open_RoundedPad1.0x1.5mm, F.Cu at (117.2, 70.0)
- added JP18: SolderJumper_3_Bridged12, Jumper:SolderJumper-3_P1.3mm_Bridged12_RoundedPad1.0x1.5mm, B.Cu at (119.1, 60.7)
- added JP19: SolderJumper_3_Bridged12, Jumper:SolderJumper-3_P1.3mm_Bridged12_RoundedPad1.0x1.5mm, B.Cu at (121.2, 54.4)
- added JP20: SolderJumper_3_Bridged12, Jumper:SolderJumper-3_P1.3mm_Bridged12_RoundedPad1.0x1.5mm, B.Cu at (96.4, 42.2)
- added JP21: SolderJumper_3_Bridged12, Jumper:SolderJumper-3_P1.3mm_Bridged12_RoundedPad1.0x1.5mm, B.Cu at (120.4, 66.8)
- added JP3: SolderJumper_2_Open, CutomParts:Jumper Connected 2 Pin Small, F.Cu at (93.5, 30.9)
- added JP7: SolderJumper_2_Open, Jumper:SolderJumper-2_P1.3mm_Open_RoundedPad1.0x1.5mm, F.Cu at (93.8, 40.8)
- added LED3: WS2812C-2020, SamacSys_Parts:WS2812C2020, F.Cu at (109.6, 60.3)
- added Q1: 40N05, Package_TO_SOT_SMD:SOT-23-3, F.Cu at (114.9, 30.8)
- added Q10: BSS138, PCM_Package_TO_SOT_SMD_AKL:SOT-23, F.Cu at (105.9, 61.9)
- added Q11: 40N05, Package_TO_SOT_SMD:SOT-23-3, F.Cu at (115.0, 45.2)
- added Q12: 40N05, Package_TO_SOT_SMD:SOT-23-3, F.Cu at (114.9, 38.1)
- added Q13: 40N05, Package_TO_SOT_SMD:SOT-23-3, F.Cu at (115.0, 48.9)
- added Q14: 40N05, Package_TO_SOT_SMD:SOT-23-3, F.Cu at (114.9, 41.6)
- added Q2: 40N05, Package_TO_SOT_SMD:SOT-23-3, F.Cu at (114.9, 34.5)
- added Q3: 40N05, Package_TO_SOT_SMD:SOT-23-3, F.Cu at (114.9, 27.2)
- added Q8: 40N05, Package_TO_SOT_SMD:SOT-23-3, F.Cu at (110.5, 50.7)
- added Q9: BSS138, PCM_Package_TO_SOT_SMD_AKL:SOT-23, F.Cu at (102.0, 61.9)
- added R29: 10, Resistor_SMD:R_0603_1608Metric, F.Cu at (111.0, 47.0)
- added R3: 10, Resistor_SMD:R_0603_1608Metric, F.Cu at (111.1, 31.1)
- added R30: 100k, Resistor_SMD:R_0402_1005Metric, F.Cu at (112.4, 38.9)
- added R31: 100k, Resistor_SMD:R_0402_1005Metric, F.Cu at (111.5, 53.9)
- added R32: 100k, Resistor_SMD:R_0402_1005Metric, F.Cu at (112.1, 42.4)
- added R33: 100k, Resistor_SMD:R_0402_1005Metric, F.Cu at (112.3, 44.7)
- added R34: 10, Resistor_SMD:R_0603_1608Metric, F.Cu at (111.1, 38.3)
- added R35: 10k, Resistor_SMD:R_0402_1005Metric, F.Cu at (111.0, 62.8)
- added R36: 120, Resistor_SMD:R_0402_1005Metric, F.Cu at (93.5, 43.4)
- added R37: 10, Resistor_SMD:R_0603_1608Metric, F.Cu at (109.6, 54.4)
- added R38: 10k, Resistor_SMD:R_0402_1005Metric, F.Cu at (108.3, 62.8)
- added R39: 10k, Resistor_SMD:R_0402_1005Metric, F.Cu at (99.7, 62.8)
- added R4: 1.5k, Resistor_SMD:R_0402_1005Metric, F.Cu at (93.7, 34.8)
- added R40: 22k, Resistor_SMD:R_0402_1005Metric, F.Cu at (119.1, 61.9)
- added R41: 10, Resistor_SMD:R_0603_1608Metric, F.Cu at (119.6, 38.9)
- added R42: 10, Resistor_SMD:R_0603_1608Metric, F.Cu at (119.6, 40.4)
- added R43: 10k, Resistor_SMD:R_0402_1005Metric, F.Cu at (119.1, 59.5)
- added R44: 100k, Resistor_SMD:R_0402_1005Metric, F.Cu at (114.5, 51.3)
- added R5: 100k, Resistor_SMD:R_0402_1005Metric, F.Cu at (112.3, 31.5)
- added R6: 10, Resistor_SMD:R_0603_1608Metric, F.Cu at (111.1, 34.7)
- added R62: 10k, Resistor_SMD:R_0402_1005Metric, F.Cu at (100.3, 64.3)
- added R63: 10k 1%, Resistor_SMD:R_0402_1005Metric, F.Cu at (109.6, 69.8)
- added R64: 10k, Resistor_SMD:R_0402_1005Metric, F.Cu at (104.9, 64.3)
- added R65: 2.2k, Resistor_SMD:R_0402_1005Metric, F.Cu at (111.0, 64.8)
- added R66: 10k, Resistor_SMD:R_0402_1005Metric, F.Cu at (118.0, 66.2)
- added R67: 4.7k, Resistor_SMD:R_0402_1005Metric, F.Cu at (119.1, 64.4)
- added R7: 100k, Resistor_SMD:R_0402_1005Metric, F.Cu at (112.4, 35.2)
- added R8: 100k, Resistor_SMD:R_0402_1005Metric, F.Cu at (112.4, 28.1)
- added R9: 10, Resistor_SMD:R_0603_1608Metric, F.Cu at (111.1, 27.8)
- added SW3: DSHP04TJGER, Button_Switch_SMD:SW_DIP_SPSTx04_Slide_Copal_CHS-04A_W5.08mm_P1.27mm_JPin, F.Cu at (115.1, 62.1)
- added U2: MOUDLE-SEEEDUINO-XIAO-ESP32C3, Arduino:ESP32-C3 16 Pin Super Mini, B.Cu at (113.7, 52.6)
- added VR1: ~, Library:EY9 reg board, B.Cu at (107.7, 44.0)
- added mouse-bite-2: VAL**, Panelization.pretty-master:mouse-bite-2mm-slot, F.Cu at (91.7, 37.3)
- added mouse-bite-4: VAL**, Panelization.pretty-master:mouse-bite-2mm-slot, F.Cu at (91.6, 63.2)
- renumbered C5 to C1, C4 to C10, C10 to C11, C2 to C12, C5 to C13, C3 to C14, C12 to C15, C1 to C2, C8 to C27, C7 to C28, C8 to C29, C4 to C3, C9 to C30, C7 to C31, C4 to C34, C5 to C35, C6 to C36, C5 to C37, C1 to C38, C4 to C39, C2 to C4, C3 to C40, C11 to C41, C6 to C42, C2 to C43, C10 to C44, C7 to C45, C8 to C46, C7 to C47, C8 to C48, C3 to C5, C6 to C7, C9 to C8, C1 to C9, D2 to D10, D1 to D2, D2 to D4, D2 to D6, D1 to D7, D1 to D8, D2 to D9, IC2 to IC10, IC4 to IC11, IC3 to IC12, IC3 to IC13, IC1 to IC3, IC2 to IC4, IC3 to IC6, IC3 to IC7, IC2 to IC9, J4 to J1, J1 to J10, J2 to J11, J8 to J12, J2 to J13, J1 to J14, J8 to J16, J7 to J2, J5 to J20, J4 to J21, J3 to J22, J15 to J23, J11 to J24, J14 to J25, J10 to J26, J6 to J27, J13 to J28, J7 to J29, J12 to J30, J9 to J31, J5 to J32, J4 to J33, J7 to J34, J6 to J35, J1 to J38, J2 to J39, J8 to J40, J2 to J41, J1 to J42, J8 to J43, J5 to J44, J6 to J45, J6 to J46, J5 to J47, J3 to J5, J7 to J6, JP2 to JP1, JP3 to JP10, JP4 to JP11, JP1 to JP13, JP1 to JP14, JP3 to JP15, JP4 to JP16, JP4 to JP17, JP1 to JP4, JP1 to JP5, JP3 to JP6, JP2 to JP8, JP2 to JP9, LED1 to LED2, LED1 to LED4, LED1 to LED5, Q2 to Q15, Q1 to Q16, Q1 to Q17, Q2 to Q18, Q1 to Q4, Q2 to Q5, Q1 to Q6, Q2 to Q7, R16 to R1, R17 to R10, R12 to R11, R8 to R12, R2 to R13, R4 to R14, R7 to R15, R17 to R16, R5 to R17, R6 to R18, R3 to R19, R16 to R2, R13 to R20, R10 to R21, R1 to R22, R12 to R23, R10 to R24, R7 to R25, R8 to R26, R13 to R27, R1 to R28, R9 to R45, R18 to R46, R2 to R47, R16 to R48, R6 to R49, R4 to R50, R18 to R51, R16 to R52, R5 to R53, R15 to R54, R14 to R55, R11 to R56, R3 to R57, R9 to R58, R11 to R59, R14 to R60, R15 to R61, R9 to R68, R17 to R69, R17 to R70, R1 to R71, R7 to R72, R8 to R73, R12 to R74, R13 to R75, R11 to R76, R14 to R77, R10 to R78, R9 to R79, R7 to R80, R12 to R81, R1 to R82, R10 to R83, R13 to R84, R8 to R85, R14 to R86, R11 to R87, R2 to R88, R3 to R89, R15 to R90, R15 to R91, R3 to R92, SW1 to SW2, SW1 to SW4, SW1 to SW5, U2 to U1, U1 to U3, U1 to U4, U1 to U5, U1 to U6, VR1 to VR2, VR1 to VR3, VR1 to VR4, VR1 to VR5, mouse-bite-2mm-slot to mouse-bite-1, mouse-bite-2mm-slot to mouse-bite-3, mouse-bite-2mm-slot to mouse-bite-5, mouse-bite-2mm-slot to mouse-bite-6, mouse-bite-2mm-slot to mouse-bite-7, mouse-bite-2mm-slot to mouse-bite-8
Routing:
- net (no net): track 3605.1 -> 4882.9 mm, vias 258 -> 383
Other:
- board size 62.2 x 94.4 mm -> 93.6 x 94.4 mm
- board text added: "4/6/25 Rev1 DAISY BOARD OUT By Will Thayer & Lucas Wilson"
- board text added: "DR6|GPIO1"
- board text added: "DR7|GPIO2"
- board text added: "DR8|GPIOA"
- board text added: "GateDrV 24V|5V"
