File: Daisy_Board_Servo/Daisy_Board_Servo.kicad_pcb (KiCad board)
At the start: 2 copper layers, 29.8 x 46.2 mm, 58 parts, among them IC1 PCA9685PW, IC2 TJA1050T_CM, IC3 LSM6DS3TR-C, J1 SM04B-SRSS-TB, J10 Conn_01x03_Pin, J11 Conn_01x03_Pin, J12 Conn_01x03_Pin, J13 Conn_01x03_Pin, J14 Conn_01x03_Pin, J15 Conn_01x03_Pin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

Commit message: Done Servo
Parts:
- added C2: 100nF 50V, Capacitor_SMD:C_0402_1005Metric, F.Cu at (91.8, 85.2)
- added C3: 100nF 50V, Capacitor_SMD:C_0402_1005Metric, F.Cu at (94.9, 90.7)
- added D3: SS34, Diode_SMD:D_SOD-123, F.Cu at (83.2, 71.1)
- added D4: ESD9XD, Diode_SMD:D_SOD-523, F.Cu at (93.6, 89.5)
- added D5: ESD9X, Diode_SMD:D_SOD-523, F.Cu at (93.5, 88.0)
- added IC4: ACS712ELCTR-05B-T, SamacSys_Parts:SOIC127P600X175-8N, F.Cu at (95.1, 83.5)
- added JP3: SolderJumper_3_Bridged12, Jumper:SolderJumper-3_P1.3mm_Bridged2Bar12_RoundedPad1.0x1.5mm, F.Cu at (94.8, 55.5)
- added JP5: SolderJumper_2_Open, Jumper:SolderJumper-2_P1.3mm_Open_RoundedPad1.0x1.5mm, B.Cu at (105.6, 78.7)
- added R24: 22k, Resistor_SMD:R_0402_1005Metric, F.Cu at (95.4, 89.2)
- added R25: 2.2k, Resistor_SMD:R_0402_1005Metric, F.Cu at (95.7, 87.7)
- added VR2: ~, Library:EY9 reg board, B.Cu at (100.7, 63.2)
- moved VR1 8.91 mm to (86.9, 74.5)
- moved C6 3.85 mm to (91.8, 83.2), turned to 90 degrees
- moved C5 3.58 mm to (84.3, 88.6)
- moved IC2 3.16 mm to (87.6, 84.4)
- moved LED1 3.14 mm to (94.2, 92.4)
- moved R10 2.58 mm to (94.3, 94.9), turned to 90 degrees
- moved R19 2.44 mm to (95.2, 78.2)
- moved R5 1.37 mm to (93.2, 79.3)
- moved R6 1.34 mm to (93.2, 78.2)
- moved R18 1.28 mm to (93.2, 77.2)
- moved D2 1.00 mm to (80.9, 71.1)
- moved C7 0.84 mm to (95.3, 96.9)
- moved R12 0.84 mm to (95.4, 94.9)
- moved R4 0.74 mm to (90.1, 80.2)
- moved C1 0.74 mm to (87.2, 80.4)
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Connections:
- J10 pad 1: GND -> ServoGND
- J11 pad 1: GND -> ServoGND
- J12 pad 1: GND -> ServoGND
- J13 pad 1: GND -> ServoGND
- J14 pad 1: GND -> ServoGND
- J15 pad 1: GND -> ServoGND
- J3 pad 1: GND -> ServoGND
- J9 pad 1: GND -> ServoGND
Routing:
- net GND: track 0.00 -> 222.9 mm, vias 0 -> 9
- net +5V: track 0.00 -> 119.8 mm, vias 0 -> 3
- net +3.3V: track 0.00 -> 92.0 mm, vias 0 -> 5
- net CANL: track 0.00 -> 60.6 mm, vias 0 -> 7
- net ServoGND: track 0.00 -> 57.2 mm
- net ServoPower: track 0.00 -> 51.3 mm
- net SCL: track 0.00 -> 40.7 mm, vias 0 -> 4
- net CANH: track 0.00 -> 38.9 mm, vias 0 -> 2
- net DipV: track 0.00 -> 36.8 mm, vias 0 -> 3
- net GPIO_1: track 0.00 -> 31.5 mm, vias 0 -> 3
- net Net-(D3-K): track 0.00 -> 30.7 mm, vias 0 -> 1
- net Net-(JP3-A): track 0.00 -> 30.5 mm, vias 0 -> 3
- net LED3: track 0.00 -> 30.0 mm, vias 0 -> 4
- net SDA: track 0.00 -> 28.8 mm, vias 0 -> 3
- net Net-(R10-Pad1): track 0.00 -> 27.6 mm, vias 0 -> 8
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- added copper zone on F.Cu, net ServoGND
- added copper zone on F.Cu, net ServoPower
Other:
- board text added: "4/9/25 Rev 1 DAISY BOARD STEP By Will Thayer & Lucas Wilson"
- board text added: "PWR"
- board text added: "VR Bridge"
- board text added: "VR2"
- board text removed: "1/14/25 Rev 3 DAISY BOARD DC By Lucas Wilson & Will Thayer"
